File: IP5306-Power-Module.kicad_sch (KiCad schematic)
At the start: 0 parts

Commit message: main
Parts:
- added C1, C2, C3: 22uF, Capacitor_SMD:C_0805_2012Metric_Pad1.18x1.45mm_HandSolder, symbol Device:C
- added C4, C5, C6, C7: 10uF, Capacitor_SMD:C_0805_2012Metric_Pad1.18x1.45mm_HandSolder, symbol Device:C
- added D1, D2, D3, D4, D5: LED, LED_SMD:LED_0603_1608Metric_Pad1.05x0.95mm_HandSolder, symbol Device:LED
- added J1: USB_C_Receptacle_USB2.0_16P, Connector_USB:USB_C_Receptacle_GCT_USB4105-xx-A_16P_TopMnt_Horizontal, symbol Connector:USB_C_Receptacle_USB2.0_16P
- added L1: L, assets:IND-SMD_L7_0-W6_6_SPM70701R0MESL_C5332207, symbol Device:L
- added R1, R2: 2R, Resistor_SMD:R_0603_1608Metric_Pad0.98x0.95mm_HandSolder, symbol Device:R
- added R3, R4: 5.1K, Resistor_SMD:R_0603_1608Metric_Pad0.98x0.95mm_HandSolder, symbol Device:R
- added R5: 20R, Resistor_SMD:R_0603_1608Metric_Pad0.98x0.95mm_HandSolder, symbol Device:R
- added R6: 10K, Resistor_SMD:R_0603_1608Metric_Pad0.98x0.95mm_HandSolder, symbol Device:R
- added SW1: KEY, Button_Switch_SMD:SW_Push_SPST_NO_Alps_SKRK, symbol Switch:SW_Push
- added U1: IP5306, assets:SOP127P600X165-9N, symbol IP5306:IP5306
Connections:
- new net: D5.2 (A), R5.2
- new net: C7.1, R2.2
- new net: C5.1, R1.2
- new net: R6.2, SW1.1
- new net BAT: C6.1, L1.2, R2.1, U1.6 (BAT)
- new net CC1: J1.A5 (CC1), R4.1
- new net CC2: J1.B5 (CC2), R3.1
- new net GND: C1.2, C2.2, C3.2, C4.2, C5.2, C6.2, C7.2, D5.1 (K), J1.A1 (GND), J1.A12 (GND), J1.B1 (GND), J1.B12 (GND), J1.SH (SHIELD), R3.2, R4.2, SW1.2, U1.9 (POWERPAD)
- new net KEY: R5.1, R6.1, U1.5 (KEY)
- new net LED1: D1.2 (A), D2.1 (K), U1.2 (LED1)
- new net LED2: D3.2 (A), D4.1 (K), U1.3 (LED2)
- new net LED3: D1.1 (K), D2.2 (A), D3.1 (K), D4.2 (A), U1.4 (LED3)
- new net SW: L1.1, U1.7 (SW)
- new net VIN: C4.1, J1.A4 (VBUS), J1.A9 (VBUS), J1.B4 (VBUS), J1.B9 (VBUS), R1.1, U1.1 (VIN)
- new net VOUT: C1.1, C2.1, C3.1, U1.8 (VOUT)
- no-connect marks 0 -> 6

Commit message: Schematic
Parts:
- added J2: S2B-XH-A_LF__SN_, assets:JST_S2B-XH-A_LF__SN_, symbol S2B-XH-A:S2B-XH-A_LF__SN_
- added J3, J4: USB_A, Connector_USB:USB_A_Molex_67643_Horizontal, symbol Connector:USB_A
Connections:
- net BAT: now also J2.1
- net GND: now also J2.2, J3.4 (GND), J3.SH (Shield), J4.4 (GND), J4.SH (Shield)
- net VOUT: now also J3.1 (VBUS), J4.1 (VBUS)
- new net: J3.2 (D-), J3.3 (D+)
- new net: J4.2 (D-), J4.3 (D+)
Other:
- moved on the sheet: C1, C2, C3, C4, C5, C6, C7, D1, D2, D3, D4, D5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

Commit message: V1
Other:
- moved on the sheet: C1, C2, C3, C4, C5, C6, C7, D1, D2, D3, D4, D5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
